File: Charging.kicad_sch (KiCad schematic)
At the start: 60 parts, among them J302 Conn_01x02_Socket, J303 2130830005, U301 SPU03L-05, U302 SPU03L-05, U303 SPU03L-05, U304 ADUM4160BRWZ, U305 USB2422T-I/MJ, U306 BQ24296RGER, U307 TPD4E1B06DRLR, U308 TPD4E1B06DRLR

Commit message: 3D models.
Parts:
- J303: Manufacturer_Part_Number (none) -> 2130830005
- U301, U302, U303: footprint SPU03L-05_MWU -> Mustang_Library:SPU03L-05_MWU; Manufacturer_Part_Number (none) -> SPU03L-05
- U304: Manufacturer_Part_Number (none) -> ADUM4160BRWZ
- U305: Manufacturer_Part_Number (none) -> USB2422T-I/MJ
- U306: Manufacturer_Part_Number (none) -> BQ24296RGER
Changed lines of the file:
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@@
 			)
 		)
-		(property "Footprint" "SPU03L-05_MWU"
+		(property "Footprint" "Mustang_Library:SPU03L-05_MWU"
 			(at 257.048 -51.816 0)
 			(effects
@@
 			)
 		)
+		(property "Manufacturer_Part_Number" "SPU03L-05"
+			(at 237.49 -58.42 0)
+			(effects
+				(font
+					(size 1.27 1.27)
+				)
+				(hide yes)
+			)
+		)
 		(pin "1"
 		)
@@
 			)
 		)
+		(property "Manufacturer_Part_Number" "BQ24296RGER"
+			(at 410.21 3.81 0)
+			(effects
+				(font
+					(size 1.27 1.27)
+				)
+				(hide yes)
+			)
+		)
 		(pin "22"
 		)
@@
 			)
 		)
-		(property "Footprint" "SPU03L-05_MWU"
+		(property "Footprint" "Mustang_Library:SPU03L-05_MWU"
 			(at 257.048 -8.636 0)
 			(effects
@@
 			)
 		)
+		(property "Manufacturer_Part_Number" "SPU03L-05"
+			(at 237.49 -15.24 0)
+			(effects
+				(font
+					(size 1.27 1.27)
+				)
+				(hide yes)
+			)
+		)
 		(pin "1"
 		)
@@
 			)
 		)
-		(property "Footprint" "SPU03L-05_MWU"
+		(property "Footprint" "Mustang_Library:SPU03L-05_MWU"
 			(at 257.048 -30.226 0)
 			(effects
@@
 			)
 		)
+		(property "Manufacturer_Part_Number" "SPU03L-05"
+			(at 237.49 -36.83 0)
+			(effects
+				(font
+					(size 1.27 1.27)
+				)
+				(hide yes)
+			)
+		)
 		(pin "1"
 		)
@@
 			)
 		)
+		(property "Manufacturer_Part_Number" "ADUM4160BRWZ"
+			(at 236.22 -104.14 0)
+			(effects
+				(font
+					(size 1.27 1.27)
+				)
+				(hide yes)
+			)
+		)
 		(pin "10"
 		)
@@
 			)
 		)
-		(property "Datasheet" "http://www.ti.com/lit/ds/symlink/tpd4e1b06.pdf"
+		(property "Datasheet" "Datasheet/tpd4e1b06.pdf"
 			(at 55.88 -144.78 0)
 			(effects
@@
 			)
 		)
-		(property "Datasheet" "USB2422T-I/MJ"
+		(property "Datasheet" "Datasheet/00001726B-3443148.pdf"
 			(at 440.436 -108.712 0)
 			(effects
@@
 			)
 		)
+		(property "Manufacturer_Part_Number" "USB2422T-I/MJ"
+			(at 506.73 -92.71 0)
+			(effects
+				(font
+					(size 1.27 1.27)
+				)
+				(hide yes)
+			)
+		)
 		(pin "3"
 		)
@@
 			)
 		)
+		(property "Manufacturer_Part_Number" "2130830005"
+			(at 119.38 -64.77 0)
+			(effects
+				(font
+					(size 1.27 1.27)
+				)
+				(hide yes)
+			)
+		)
 		(pin "SH4"
 		)
@@
 			)
 		)
-		(property "Datasheet" "http://www.ti.com/lit/ds/symlink/tpd4e1b06.pdf"
+		(property "Datasheet" "Datasheet/tpd4e1b06.pdf"
 			(at 53.34 -88.9 0)
 			(effects

Commit message: Place and align PCB components to enclosure DXF. Expand PCB 15mm both sides of USB-C. Move BM83 to right side. Cutout PCB along right side for antenna function.
Parts:
- removed J302: Conn_01x02_Socket, Mustang_Library:BatteryHolder_Keystone_1042_1x18650, symbol Mustang_Library:Conn_01x02_Socket
- added C1: 0.1uF, Mustang_Library:C_0805_2012Metric_Pad1.18x1.45mm_HandSolder, symbol Mustang_Library:CAP_CERAMIC0805-NOOUTLINE
- added C2, C3: 1uF, Mustang_Library:C_0805_2012Metric_Pad1.18x1.45mm_HandSolder, symbol Mustang_Library:C
- added C4, C5: 18pF, Mustang_Library:C_0805_2012Metric_Pad1.18x1.45mm_HandSolder, symbol Mustang_Library:CAP_CERAMIC0805-NOOUTLINE
- added J3: Conn_01x02_Pin, Mustang_Library:JST_PH_S2B-PH-K_1x02_P2.00mm_Horizontal, symbol Mustang_Library:Conn_01x02_Pin
- added R1: 100k, Mustang_Library:R_0805_2012Metric_Pad1.20x1.40mm_HandSolder, symbol Mustang_Library:R
- added R2: 100k, Mustang_Library:R_0805_2012Metric_Pad1.20x1.40mm_HandSolder, symbol Mustang_Library:RESISTOR0805_NOOUTLINE
- added R3: 12k, Mustang_Library:R_0805_2012Metric_Pad1.20x1.40mm_HandSolder, symbol Mustang_Library:R
- added R4, R5, R6, R7: 24R, Mustang_Library:R_0805_2012Metric_Pad1.20x1.40mm_HandSolder, symbol Mustang_Library:RESISTOR0805_NOOUTLINE
- added Y1: 25MHz, symbol Mustang_Library:Crystal
- U302: symbol Mustang_Library:SPU03L-05_2 -> Mustang_Library:SPU03L-05_2_2
- U303: symbol Mustang_Library:SPU03L-05_2 -> Mustang_Library:SPU03L-05_2_1
- U305: Manufacturer_Part_Number USB2422T-I/MJ -> (none)
Connections:
- net EPAD is gone; now on net GND: U305.25 (EPAD)
- net USCL is gone; now on net SCL: R326.1
- net USDA is gone; now on net SDA: R327.1
- net 3V3: now also C1.1, C2.1
- net BAT: now also J3.1 (Pin_1)
- net CRFILT: now also C3.1
- net Earth: no longer J303.SH1 (SHIELD1), J303.SH2 (SHIELD2), J303.SH3 (SHIELD3), J303.SH4 (SHIELD4)
- net GND: now also C1.2, C2.2, C3.2, C4.1, C5.1, J3.2 (Pin_2), R1.2, R3.1
- net GNDPWR: now also J303.SH1 (SHIELD1), J303.SH2 (SHIELD2), J303.SH3 (SHIELD3), J303.SH4 (SHIELD4)
- net RBIAS: now also R3.2
- net SCL: no longer R315.2, R326.2, U306.5 (SCL)
- net SDA: no longer R316.2, R327.2, U306.6 (SDA)
- net SMBCLK: now also R4.2
- net SMBDATA: now also R6.2
- net VBUS_DET: now also R1.1, R2.2
- net XIN: now also C4.2, Y1.2
- net XOUT: now also C5.2, Y1.1
- net SUSP renamed SUSP_IND
- net SUSP_IND: now also R7.2
- net UCE renamed BQCE
- net UINT renamed BQINT
- net UOTG renamed BQOTG
- net UPG renamed BQPG
- net UPSEL renamed BQPSEL
- net UQON renamed BQQON
- net USTAT renamed BQSTAT
- net VBUS-U6 renamed VBUS-ISO
- net VBUS-ISO: now also R2.1
- net /OCS1 renamed OCS1_N
- net /OCS2 renamed OCS2_N
- net /RESET renamed _RESET_N
- net _RESET_N: now also R5.2
- new net USBRESET_N: R5.1
- new net USBSMBCLK: R4.1
- new net USBSMBDATA: R6.1
- new net USBSUSP_IND: R7.1
- new net _SCL: R315.2, R326.2, U306.5 (SCL)
- new net _SDA: R316.2, R327.2, U306.6 (SDA)
Other:
- moved on the sheet: C301, C302, C303, C304, C305, C306, C307, C308, C309, C310, C311, C312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

Commit message: Electrical Rules Check fixes in progress.
Parts:
- removed J3: Conn_01x02_Pin, Mustang_Library:JST_PH_S2B-PH-K_1x02_P2.00mm_Horizontal, symbol Mustang_Library:Conn_01x02_Pin
- removed R301, R302, R303, R304, R305, R306, R307, R308, R319, R320, R321, R322, R323, R324, R325, R326, R327, R4, R5, R6, R7: 24R, Mustang_Library:R_0805_2012Metric_Pad1.20x1.40mm_HandSolder, symbol Mustang_Library:RESISTOR0805_NOOUTLINE
- added C10, C11, C6: 0.1uF, Mustang_Library:C_0805_2012Metric_Pad1.18x1.45mm_HandSolder, symbol Mustang_Library:CAP_CERAMIC0805-NOOUTLINE
- added J3: Conn_01x02_Pin_JST-PH_Batt, Mustang_Library:JST_PH_S2B-PH-K_1x02_P2.00mm_Horizontal, symbol Mustang_Library:Conn_01x02_Pin_JST-PH_Batt
- added R12, R8, R9: 0R, symbol Mustang_Library:R_h
- added R16, R17, R18, R19, R301, R302, R303, R304, R305, R306, R307, R308, R319, R320, R321, R322, R323, R324, R325, R326, R327, R4, R5, R6, R7: 24R, symbol Mustang_Library:R_h
- U301: symbol Mustang_Library:SPU03L-05_2 -> Mustang_Library:SPU03L-05
- U302: symbol Mustang_Library:SPU03L-05_2_2 -> Mustang_Library:SPU03L-05
- U303: symbol Mustang_Library:SPU03L-05_2_1 -> Mustang_Library:SPU03L-05
Connections:
- net NC307 is gone; now on net GNDPWR: U307.5 (NC)
- net NC308 is gone; now on net GNDPWR: U308.5 (NC)
- net _SCL is gone; now on net SCL: R315.2, U306.5 (SCL)
- net _SDA is gone; now on net SDA: R316.2, U306.6 (SDA)
- net BAT: now also R8.1
- net CE: now also R320.2
- net DD+: now also R304.1
- net DD-: now also R303.1
- net DM1: now also R16.1
- net DM2: now also R18.1
- net DMU: now also R303.2
- net DP1: now also R17.1
- net DP2: now also R19.1
- net DPU: now also R304.2
- net GND: now also C10.2, C11.2, C6.2, R9.1
- net GNDPWR: now also R12.1; no longer J303.SH1 (SHIELD1), J303.SH2 (SHIELD2), J303.SH3 (SHIELD3), J303.SH4 (SHIELD4)
- net INT: now also R325.2
- net OTG: now also R321.2
- net PDEN: now also R306.2
- net PG: now also R323.2
- net PIN: now also R308.1
- net PSEL: now also R322.2
- net QON: now also R319.2
- net SCL: now also R326.2
- net SDA: now also R327.2
- net SMBCLK: now also R4.2
- net SMBDATA: now also R5.2
- net SPD: now also R307.1
- net SPU: now also R305.2
- net STAT: now also R324.2
- net SUSP_IND: now also R7.2
- net UD+: now also R302.2
- net UD-: now also R301.2
- net VDD1: now also R305.1, R306.1
- net 3V3 renamed +3V3
- net +3V3: now also R307.2, R308.2
- net DA+ renamed DAB+
- net DAB+: now also R302.1
- net DB- renamed DAB-
- net DAB-: now also R301.1
- net VBUS-ISO renamed 5V
- net 5V: now also C6.1
- net _RESET_N renamed RESET_N
- net RESET_N: now also R6.2
- new net: J303.SH1 (SHIELD1), J303.SH2 (SHIELD2), J303.SH3 (SHIELD3), J303.SH4 (SHIELD4), R12.2
- new net +BATT: C11.1, J3.1 (+Batt), R8.2
- new net -BATT: C10.1, J3.2 (-Batt), R9.2
- new net BAT_CE: R320.1
- new net BAT_INT: R325.1
- new net BAT_OTG: R321.1
- new net BAT_PG: R323.1
- new net BAT_PSEL: R322.1
- new net BAT_QON: R319.1
- new net BAT_SCL: R326.1
- new net BAT_SDA: R327.1
- new net BAT_STAT: R324.1
- new net USB_DM_BT: R18.2
- new net USB_DM_MCU: R16.2
- new net USB_DP_BT: R19.2
- new net USB_DP_MCU: R17.2
- new net USB_RESET_N: R6.1
- new net USB_SMBCLK: R4.1
- new net USB_SMBDATA: R5.1
- new net USB_SUSP_IND: R7.1
Other:
- moved on the sheet: C304, C305, C306, C307, C308, C309, C310, C311, C312, L301, L302, L303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

Commit message: wip
Parts:
- added C12, C13: 1uF, Mustang_Library:C_0805_2012Metric_Pad1.18x1.45mm_HandSolder, symbol Mustang_Library:C
- added U4: LP5907MFX-3.3_NOPB, Mustang_Library:SOT95P280X145-5N, symbol LP5907MFX-3.3:LP5907MFX-3.3_NOPB
Connections:
- net +3V3: now also C13.1, U4.5 (OUT)
- net GND: now also C12.2, C13.2, U4.2 (GND)
- net VSYS: now also C12.1, U4.1 (IN), U4.3 (EN)

Commit message: wip
Parts:
- added C20, C21, C26: 0.1uF, Mustang_Library:C_0805_2012Metric_Pad1.18x1.45mm_HandSolder, symbol Mustang_Library:CAP_CERAMIC0805-NOOUTLINE
- added D10: EAST1616RGBA3, Mustang_Library:LED_EAST1616RGBA3, symbol Mustang_Library:EAST1616RGBA3
- added R70, R81, R82, R83: 24R, symbol Mustang_Library:R_h
- added R84, R85, R86: 5.1K, symbol Mustang_Library:R_h
- added R87, R88, R89: 0R, symbol Mustang_Library:R_h
- R305, R306, R307, R308: value 24R -> 10K
Connections:
- net +3V3: now also C21.1, D10.3, R88.2, R89.2; no longer C303.2, R307.2, R308.2, U304.14 (VDD2), U304.16 (VBUS2)
- net BAT_PG: now also R84.1
- net BAT_STAT: now also R85.1
- net GND: now also C20.2, C21.2, C26.1
- net OCS1_N: now also R81.1
- net OCS2_N: now also R83.1
- net PRTPWR1: now also R70.1
- net PRTPWR2: now also R82.1
- net +BATT: no longer names the net of C11.1, J3.1 (+Batt), R8.2
- net -BATT: no longer names the net of C10.1, J3.2 (-Batt), R9.2
- net 5V renamed VUSB
- net VUSB: now also R87.2
- net BAT renamed VBATT
- net NC: no longer names the net of U305.6 (NC)
- net PLLFILT: no longer names the net of U305.23 (PLLFILT)
- net PLLFILT: now also C20.1
- new net: C26.2, R87.1, R88.1, U304.16 (VBUS2)
- new net: C303.2, R307.2, R308.2, R89.1, U304.14 (VDD2)
- new net: D10.4, R84.2
- new net: D10.2, R85.2
- new net: D10.1, R86.2
- no-connect marks 0 -> 5
Other:
- moved on the sheet: C12, C13, C303, U4

Commit message: Use all YAGEO 0603 resistors.
Parts:
- added R90: 24R, Mustang_Library:R_0603_1608Metric, symbol Mustang_Library:R_0603_24R
- R1: value 100k -> 100K; footprint Mustang_Library:R_0805_2012Metric_Pad1.20x1.40mm_HandSolder -> Mustang_Library:R_0603_1608Metric; symbol Mustang_Library:R -> Mustang_Library:R_0603_100K; MPN (none) -> AC0603FR-07100KL; Manufacturer (none) -> Yageo; Power (none) -> .1W
- R12, R8, R87, R88, R89, R9: footprint (none) -> Mustang_Library:R_0603_1608Metric; symbol Mustang_Library:R_h -> Mustang_Library:R_0603_0R; MPN (none) -> AC0603JR-070RL; Manufacturer (none) -> Yageo; Power (none) -> J
- R16, R17, R18, R19, R301, R302, R303, R304, R319, R320, R321, R322, R323, R324, R325, R326, R327, R4, R5, R6, R7, R70, R81, R82, R83: footprint (none) -> Mustang_Library:R_0603_1608Metric; symbol Mustang_Library:R_h -> Mustang_Library:R_0603_24R; MPN (none) -> AC0603JR-0724RL; Manufacturer (none) -> Yageo; Power (none) -> .1W
- R2: value 100k -> 100K; footprint Mustang_Library:R_0805_2012Metric_Pad1.20x1.40mm_HandSolder -> Mustang_Library:R_0603_1608Metric; symbol Mustang_Library:RESISTOR0805_NOOUTLINE -> Mustang_Library:R_0603_100K; MPN (none) -> AC0603FR-07100KL; Manufacturer (none) -> Yageo; Power (none) -> .1W
- R3: value 12k -> 12K; footprint Mustang_Library:R_0805_2012Metric_Pad1.20x1.40mm_HandSolder -> Mustang_Library:R_0603_1608Metric; symbol Mustang_Library:R -> Mustang_Library:R_0603_12K; MPN (none) -> AC0603FR-0712KL; Manufacturer (none) -> Yageo; Power (none) -> .1W
- R305, R306, R307, R308: footprint (none) -> Mustang_Library:R_0603_1608Metric; symbol Mustang_Library:R_h -> Mustang_Library:R_0603_10K; MPN (none) -> AC0603FR-7W10KL; Manufacturer (none) -> Yageo; Power (none) -> .2W
- R309: value 31.23k -> 30.9K; footprint Mustang_Library:R_0805_2012Metric_Pad1.20x1.40mm_HandSolder -> Mustang_Library:R_0603_1608Metric; symbol Mustang_Library:R -> Mustang_Library:R_0603_30.9K; MPN (none) -> AC0603FR-0730K9L; Manufacturer (none) -> Yageo; Power (none) -> .1W
- R310: value 5.25k -> 5.23K; footprint Mustang_Library:R_0805_2012Metric_Pad1.20x1.40mm_HandSolder -> Mustang_Library:R_0603_1608Metric; symbol Mustang_Library:R -> Mustang_Library:R_0603_5.23K; MPN (none) -> AC0603FR-075K23L; Manufacturer (none) -> Yageo; Power (none) -> .1W
- R311: value 250R -> 249R; footprint Mustang_Library:R_0805_2012Metric_Pad1.20x1.40mm_HandSolder -> Mustang_Library:R_0603_1608Metric; symbol Mustang_Library:R -> Mustang_Library:R_0603_249R; MPN (none) -> AC0603JR-07249RL; Manufacturer (none) -> Yageo; Power (none) -> .1W
- R312, R313, R314, R315, R316: value 10k -> 10K; footprint Mustang_Library:R_0805_2012Metric_Pad1.20x1.40mm_HandSolder -> Mustang_Library:R_0603_1608Metric; symbol Mustang_Library:R -> Mustang_Library:R_0603_10K; MPN (none) -> AC0603FR-7W10KL; Manufacturer (none) -> Yageo; Power (none) -> .2W
- R317, R318: value 5.1k -> 5.23K; footprint Mustang_Library:R_0805_2012Metric_Pad1.20x1.40mm_HandSolder -> Mustang_Library:R_0603_1608Metric; symbol Mustang_Library:RESISTOR0805_NOOUTLINE -> Mustang_Library:R_0603_5.23K; MPN (none) -> AC0603FR-075K23L; Manufacturer (none) -> Yageo; Power (none) -> .1W
- R84, R85, R86: value 5.1K -> 5.23K; footprint (none) -> Mustang_Library:R_0603_1608Metric; symbol Mustang_Library:R_h -> Mustang_Library:R_0603_5.23K; MPN (none) -> AC0603FR-075K23L; Manufacturer (none) -> Yageo; Power (none) -> .1W
- U307, U308: Link https://www.ti.com/lit/ds/symlink/tpd4e1b06.pdf -> (none)
Connections:
- net +3V3: no longer R312.1, R313.1, R314.1, R315.1, R316.1
- net BAT_INT: now also R86.1
- net CC1: now also R318.1; no longer R318.2
- net GND: now also R1.1, R3.2, U305.6 (NC), U4.4; no longer R1.2, R3.1
- net GNDPWR: now also R318.2; no longer R318.1
- net INT: no longer R314.2
- net PG: no longer R312.2
- net RBIAS: now also R3.1; no longer R3.2
- net SCL: no longer R315.2
- net SDA: no longer R316.2
- net STAT: no longer R313.2
- net VBUS_DET: now also R1.2; no longer R1.1
- net VSYS: now also R90.1; no longer U4.3 (EN)
- new net: R90.2, U4.3 (EN)
- no-connect marks 5 -> 4
Other:
- moved on the sheet: R1, R3, R309, R310, R311, TH301
