File: mcu.kicad_sch (KiCad schematic)
At the start: 0 parts

Commit message: Place and align PCB components to enclosure DXF. Expand PCB 15mm both sides of USB-C. Move BM83 to right side. Cutout PCB along right side for antenna function.
Parts:
- added J4: Micro_SD_Card_4.0_CUI, Mustang_Library:microSD_XC_CUI_MSD4-1-A, symbol Mustang_Library:Micro_SD_Card_4.0_CUI
- added U3: STM32L496VGTx, Mustang_Library:LQFP-100_14x14mm_P0.5mm, symbol Mustang_Library:STM32L496VGTx
Connections:
- new net GND: U3.10 (VSS), U3.19 (VSSA), U3.27 (VSS), U3.49 (VSS), U3.74 (VSS), U3.99 (VSS)

Commit message: Electrical Rules Check fixes in progress.
Parts:
- added R15: 0R, symbol Mustang_Library:R_h
Connections:
- net GND: now also R15.1
- net at J4.10 (SHIELD): now also J4.11 (SHIELD), J4.12 (SHIELD), J4.13 (SHIELD), J4.14 (SHIELD), R15.2
- no-connect marks 0 -> 38

Commit message: Use all YAGEO 0603 resistors.
Parts:
- added C29, C30, C31, C32, C33, C34, C35, C36: 0.1uF, Mustang_Library:C_0805_2012Metric_Pad1.18x1.45mm_HandSolder, symbol Mustang_Library:CAP_CERAMIC0805-NOOUTLINE
- added C37, C38, C39, C40, C41: 1uF, Mustang_Library:C_0805_2012Metric_Pad1.18x1.45mm_HandSolder, symbol Mustang_Library:C
- added R100, R101, R102, R103, R104, R105, R106, R107, R108, R109, R110, R111, R112, R113, R114, R115, R97, R98, R99: 24R, Mustang_Library:R_0603_1608Metric, symbol Mustang_Library:R_0603_24R
- added R95: 0R, Mustang_Library:R_0603_1608Metric, symbol Mustang_Library:R_0603_0R
- added U10, U11, U6, U9: TPD4E1B06DRLR, Mustang_Library:SOTFL50P160X60-6N, symbol Mustang_Library:TPD4E1B06DRLR
- added U7: LP5907MFX-3.3_NOPB, Mustang_Library:SOT95P280X145-5N, symbol LP5907MFX-3.3:LP5907MFX-3.3_NOPB
- added U8: LP5907MFX-1.8_NOPB, Mustang_Library:SOT95P280X145-5N, symbol LP5907MFX-3.3:LP5907MFX-1.8_NOPB
- R15: footprint (none) -> Mustang_Library:R_0603_1608Metric; symbol Mustang_Library:R_h -> Mustang_Library:R_0603_0R; MPN (none) -> AC0603JR-070RL; Manufacturer (none) -> Yageo; Power (none) -> J
- U3: value STM32L496VGTx -> STM32L496VGT6_Mustang; footprint Mustang_Library:LQFP-100_14x14mm_P0.5mm -> Package_QFP:LQFP-100_14x14mm_P0.5mm; symbol Mustang_Library:STM32L496VGTx -> Mustang_Library:STM32L496VGT6_Mustang
Connections:
- net GND: now also J4.17 (VSS), J4.20 (VSS), J4.21 (D1-), J4.23 (VSS), J4.6 (VSS), C29.2, C30.2, C31.2, C32.2, C33.2, C34.2, C35.2, C36.2, C37.2, C38.2, C39.2, C40.2, C41.2, R101.2, U10.2 (GND), U10.5 (NC), U11.2 (GND), U11.5 (NC), U6.2 (GND), U6.3 (IO2), U6.5 (NC), U7.2 (GND), U7.4, U8.2 (GND), U8.4, U9.2 (GND), U9.5 (NC)
- net USB_RESET_N: now also R114.2
- net USB_SUSP_IND: now also R115.2
- net VSYS: now also C38.1, C40.1, U7.1 (IN), U8.1 (IN)
- net at J4.1 (DAT2): now also R105.2, U10.6 (IO4)
- net at J4.15 (VDD_1.8): now also C41.1, U11.1 (IO1), U8.5 (OUT)
- net at J4.16 (SWIO): now also R100.2, U9.1 (IO1)
- net at J4.18 (D0+): now also R109.2, U6.6 (IO4)
- net at J4.19 (D0-): now also R110.2, U6.4 (IO3)
- net at J4.2 (DAT3/CD): now also R106.2, U10.4 (IO3)
- net at J4.22 (D1+): now also R102.2, U6.1 (IO1)
- net at J4.3 (CMD): now also R108.1, U10.3 (IO2)
- net at J4.4 (VDD_3.3): now also C39.1, U11.3 (IO2), U7.5 (OUT)
- net at J4.5 (CLK): now also R107.2, U10.1 (IO1)
- net at J4.7 (DAT0/RCLK+): now also R103.2, U9.6 (IO4)
- net at J4.8 (DAT1/RCLK-): now also R104.2, U9.4 (IO3)
- net at J4.9 (CD): now also R99.2, U9.3 (IO2)
- net +3V3: now reaches U3.100 (VDD)
- net +3V3: now also U3.11 (VDD), U3.28 (VDD), U3.50 (VDD), U3.75 (VDD), C31.1, C32.1, C33.1, C34.1, C35.1, R95.1
- net at U3.17 (PC2): now also R97.1
- net at U3.18 (PC3): now also R98.1
- net at U3.22 (VDDA): now also C30.1, C37.1, R95.2
- net at U3.33 (PC4): now also R99.1
- net at U3.34 (PC5): now also R100.1
- net VBAT: now reaches U3.6 (VBAT)
- net VBAT: now also C36.1
- net at U3.63 (PC6): now also R101.1
- net at U3.64 (PC7): now also R102.1
- net at U3.65 (PC8): now also R103.1
- net at U3.66 (PC9): now also R104.1
- net at U3.67 (PA8): now also R115.1
- net at U3.68 (PA9): now also R114.1
- net at U3.69 (PA10): now also R111.1
- net USB_DM: now reaches U3.70 (PA11)
- net USB_DP: now reaches U3.71 (PA12)
- net at U3.72 (PA13): now also R112.1
- net VUSB: now reaches U3.73 (VDDUSB)
- net VUSB: now also C29.1
- net at U3.76 (PA14): now also R113.1
- net at U3.78 (PC10): now also R105.1
- net at U3.79 (PC11): now also R106.1
- net at U3.80 (PC12): now also R107.1
- net at U3.83 (PD2): now also R108.2
- net at U3.95 (PB8): now also R109.1
- net at U3.96 (PB9): now also R110.1
- new net: R97.2, U7.3 (EN)
- new net: R98.2, U8.3 (EN)
- no-connect marks 38 -> 39
Other:
- moved on the sheet: J4, R15
